File: HW/SWD_Isolator.kicad_pcb (KiCad board)
At the start: 2 copper layers, 30.1 x 12.8 mm, 17 parts, among them J1 Conn_01x05_Male, J2 Conn_01x05_Male, U1 Si8645BB-B-IS1

Commit message: Update to Rev2
Parts:
- J1: value Conn_01x05_Male -> Conn_01x05
- J2: value Conn_01x05_Male -> Conn_01x05; footprint Connector_PinSocket_2.54mm:PinSocket_1x05_P2.54mm_Horizontal -> Connector_PinHeader_2.54mm:PinHeader_1x05_P2.54mm_Horizontal
- U1: value Si8645BB-B-IS1 -> SI8605AC
- moved J2 10.2 mm to (95.0, 38.3), turned to 0 degrees
- moved J1 0.46 mm to (72.1, 48.5)
- moved U1 0.05 mm to (83.6, 43.4)
- renumbered R3 to R2, R2 to R3
Connections:
- C1 pad 2: GND -> GND1
- C2 pad 2: GND -> GND1
- C3 pad 2: GNDA -> GND2
- C4 pad 2: GNDA -> GND2
- D1 pad 1: GND -> GND1
- D2 pad 1: GNDA -> GND2
- J1 pad 2: GND -> GND1
- J2 pad 1: VDD -> Net-(J2-Pad1)
- J2 pad 2: GNDA -> Net-(J2-Pad2)
- J2 pad 4: Net-(J2-Pad4) -> GND2
- J2 pad 5: Net-(J2-Pad5) -> VDD
- R4 pad 2: Net-(J2-Pad4) -> Net-(J2-Pad2)
- R5 pad 2: Net-(J2-Pad5) -> Net-(J2-Pad1)
- U1 pad 10: Net-(U1-Pad10) -> (no net)
- U1 pad 11: Net-(J2-Pad5) -> Net-(J2-Pad1)
- U1 pad 14: Net-(J2-Pad4) -> Net-(J2-Pad2)
- U1 pad 15: GNDA -> (no net)
- U1 pad 2: GND -> (no net)
- U1 pad 5: Net-(U1-Pad5) -> (no net)
- U1 pad 7: Net-(U1-Pad7) -> (no net)
- U1 pad 8: GND -> GND1
- U1 pad 9: GNDA -> GND2
Routing:
- net Net-(J2-Pad5): track 20.6 -> 0.00 mm, vias 4 -> 0
- net Net-(J2-Pad1): track 0.00 -> 20.6 mm, vias 0 -> 4
- net Net-(J2-Pad4): track 14.6 -> 0.00 mm
- net Net-(J2-Pad2): track 0.00 -> 14.6 mm
- net GND1: track 0.00 -> 12.1 mm, vias 0 -> 12
- net GND: track 12.1 -> 0.00 mm, vias 12 -> 0
- net GNDA: track 12.0 -> 0.00 mm, vias 9 -> 0
- net GND2: track 0.00 -> 12.0 mm, vias 0 -> 9
- added copper zone on B.Cu, net GND1
- added copper zone on F.Cu, net GND1
- added copper zone on B.Cu, net GND2
- added copper zone on F.Cu, net GND2
- removed copper zone on B.Cu, net GND
- removed copper zone on F.Cu, net GND
- removed copper zone on B.Cu, net GNDA
- removed copper zone on F.Cu, net GNDA
Other:
- board size 30.1 x 12.8 mm -> 30 x 12.8 mm
- board text added: "->"
- board text added: "<->"
- board text added: "SWD, I2C, UART ISOLATOR"
- board text removed: "SWD & I2C ISOLATOR"
